File: linear-dimmer.kicad_pcb (KiCad board)
At the start: 2 copper layers, 49.3 x 30.4 mm, 31 parts, among them CON1 BARREL_JACK, P1 POWER, Q1 BUK6207-55C, SW1 Switch_SPDT_x2, U1 LM78L05ACZ, U2 MCP6072, U3 REF3012, U4 MCP65R41T

Commit message: Add amperage markings
Other:
- board text added: "0.9A"
- board text added: "1.8A"
Changed lines of the file:
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@@
     (area 109.826697 69.920466 159.226699 100.420468)
     (thickness 1.6)
-    (drawings 34)
+    (drawings 36)
     (tracks 583)
     (zones 0)
@@
     )
   )
+  (gr_text 1.8A (at 144.6 70.8) (layer B.SilkS)
+    (effects (font (size 0.7 0.7) (thickness 0.15)) (justify mirror))
+  )
+  (gr_text 0.9A (at 137.1 70.8) (layer B.SilkS)
+    (effects (font (size 0.7 0.7) (thickness 0.15)) (justify mirror))
+  )
   (gr_text "LED dimmer v2.0\nciobreliai.lt \ntechnariumas.lt\n\nmic@wemakethings.net\n2015" (at 150.25 85.25 270) (layer B.SilkS)

Commit message: Fix version number on silkscreen
Other:
- board text added: "LED dimmer v2.1 ciobreliai.lt technariumas.lt mic@wemakethings.net 2015"
- board text removed: "LED dimmer v2.0 ciobreliai.lt technariumas.lt mic@wemakethings.net 2015"
Changed lines of the file:
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@@
-(kicad_pcb (version 4) (host pcbnew 0.201511161334+6316~30~ubuntu14.04.1-product)
+(kicad_pcb (version 4) (host pcbnew 0.201511300701+6336~38~ubuntu14.04.1-stable)
   (general
     (links 64)
@@
     (effects (font (size 0.7 0.7) (thickness 0.15)) (justify mirror))
   )
-  (gr_text "LED dimmer v2.0\nciobreliai.lt \ntechnariumas.lt\n\nmic@wemakethings.net\n2015" (at 150.25 85.25 270) (layer B.SilkS)
+  (gr_text "LED dimmer v2.1\nciobreliai.lt \ntechnariumas.lt\n\nmic@wemakethings.net\n2015" (at 150.25 85.25 270) (layer B.SilkS)
     (effects (font (size 1.5 1.5) (thickness 0.3)) (justify mirror))
   )
